File: hw/sch_pcb/PIND02.kicad_sch (KiCad schematic)
At the start: 58 parts, among them J1 Conn_Coaxial, J2 MLAB I2C interface, J3 HEADER_2x01, M1 HOLE M3, M2 HOLE M3, M3 HOLE, M4 HOLE, M5 RFShield_TwoPieces, Q1 2SK2394-6, U1 OPA2314, U3 ISL21080DIH312Z-TK, U3 SHT31-DIS, U4 TPS613222ADBV

Commit message: Update measured values.
Other:
- note added: "+317 uA"
- note added: "1.5 V @ 5V VDD 1.48 V @ 3.3V VDD"
- note added: "149 mV"
- note removed: "+403 uA"
- note removed: "1.89 V"
Changed lines of the file:
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@@
     (stroke (width 0) (type default))
   )
-  (text "+403 uA" (at 73.66 78.486 0)
+  (text "+317 uA" (at 73.66 78.486 0)
     (effects (font (size 1.524 1.524)) (justify left bottom))
   )
@@
     (effects (font (size 1.524 1.524)) (justify left bottom))
   )
-  (text "1.89 V" (at 90.17 97.536 0)
+  (text "1.5 V @ 5V VDD\n1.48 V @ 3.3V VDD" (at 63.5 93.98 0)
     (effects (font (size 1.524 1.524)) (justify left bottom))
   )
   (text "+" (at 74.93 114.3 90)
     (effects (font (size 1.524 1.524)) (justify right bottom))
+  )
+  (text "149 mV" (at 125.73 62.23 0)
+    (effects (font (size 1.524 1.524)) (justify left bottom))
   )
   (text "Noise filtering" (at 73.66 123.19 0)
@@
   (symbol (lib_id "MLAB_T:Q_NJFET_SDG") (at 90.17 82.55 0) (mirror y) (unit 1)
     (in_bom yes) (on_board yes) (dnp no) (fields_autoplaced)
-    (property "Reference" "Q1" (at 85.09 81.2798 0)
-      (effects (font (size 1.27 1.27)) (justify left))
-    )
-    (property "Value" "2SK2394-6" (at 85.09 83.8198 0)
+    (property "Reference" "Q1" (at 85.09 81.28 0)
+      (effects (font (size 1.27 1.27)) (justify left))
+    )
+    (property "Value" "2SK2394-6" (at 85.09 83.82 0)
       (effects (font (size 1.27 1.27)) (justify left))
     )
@@
       (effects (font (size 1.27 1.27)) hide)
     )
-    (property "Datasheet" "~" (at 90.17 82.55 0)
-      (effects (font (size 1.27 1.27)) hide)
-    )
+    (property "Datasheet" "https://cz.mouser.com/datasheet/2/308/1/2SK2394_D-3150134.pdf" (at 90.17 82.55 0)
+      (effects (font (size 1.27 1.27)) hide)
+    )
